File: ledriver_pcb/ledriver_pcb.sch (KiCad schematic (older format))
At the start: 43 parts, among them J1 5-12vdc, J10 POT2, J11 I2C, J12 Serial2, J13 Serial1, J14 M3, J15 M3, J16 M3, J17 M3, J2 USB_B, J3 USB+-, J4 USB_EXT, J5 RJ2, J6 CONN-114-00841-68-MICROSD, J7 RJ1, J8 led_out_clk, J9 POT1, SW1 SW_SPST, SW2 SW_SPST, SW3 SW_SPST, U1 L7805, U2 MCP1825, U3 WIZ820IO, U4 74HC245, U5 Teensy3.2

Commit message: changed led SPI output to use pin 7 and 14, not reflected in layout
Parts:
- removed J10: POT2, Potentiometers:Potentiometer_Bourns_PTV09A-1_Horizontal, symbol Conn_01x03
- removed J9: POT1, Potentiometers:Potentiometer_Bourns_PTV09A-1_Horizontal, symbol Conn_01x03
- added C7: C, Capacitors_SMD:C_0603_HandSoldering, symbol C
- added D4: WS2812B, SparkFun-LED:WS2812B, symbol WS2812B
- added J18: Serial3, Connectors_Molex:Molex_KK-6410-04_04x2.54mm_Straight, symbol Conn_01x04
- added J19: underglow, Connectors:GS2, symbol GS2
- added R3: 4K, Resistors_SMD:R_0603_HandSoldering, symbol R
- added RV1, RV2: POT, Potentiometers:Potentiometer_Bourns_PTV09A-1_Horizontal, symbol POT
- added SW4: SW_SPST, Buttons_Switches_THT:SW_Tactile_SPST_Angled_PTS645Vx39-2LFS, symbol SW_SPST
- U4: footprint Housings_SSOP:SSOP-20_5.3x7.2mm_Pitch0.65mm -> Housings_SOIC:SOIC-20W_7.5x12.8mm_Pitch1.27mm
Connections:
- net labels added: RX3, TX3
- wire segments 183 -> 164
- no-connect marks 37 -> 38
Other:
- note added: "BACK"
- note added: "DOWN"
- note added: "SELECT"
- note added: "UP"
- note added: "now uses pin 7 and 14 for SPI output for APA102"
- note added: "put it on the underside!!! underglow"
- note removed: "use as clock line for ws2801"
- moved on the sheet: R9

Commit message: swapping a few pins to fix ehternet SPI CS thing
Connections:
- wire segments 164 -> 163
Other:
- note added: "status went from pin 22 to pin 3\nbuttons to pin 22\nwiz CS to 15"
Changed lines of the file:
@@
 Text Label 12200 2700 2    60   ~ 0
 SPI_DIN
-Text Label 12200 1900 2    60   ~ 0
+Text Label 12200 3500 2    60   ~ 0
 SPI_CS_WIZ
 Text Label 12200 3300 2    60   ~ 0
@@
 Text Label 14200 3800 0    60   ~ 0
 WIZ_RESET
-Text Label 12200 1800 2    60   ~ 0
+Text Label 12200 1900 2    60   ~ 0
 SPI_CS_SDCARD
 Text Label 11450 2400 2    60   ~ 0
@@
 Text Label 8850 6650 2    60   ~ 0
 I2C_SDA
-Text Label 11450 3500 2    60   ~ 0
+Text Label 11450 3600 2    60   ~ 0
 POT1
-Text Label 11450 3600 2    60   ~ 0
+Text Label 11450 3700 2    60   ~ 0
 POT2
-Text Label 11450 3700 2    60   ~ 0
+Text Label 14200 3900 0    60   ~ 0
 BUTTONS
 Text Label 9500 5600 2    60   ~ 0
@@
 	0    1    1    0
 $EndComp
-Text Label 14200 3900 0    60   ~ 0
+Text Label 12200 1800 2    60   ~ 0
 STATUS
 $Comp
@@
 	9600 4200 9600 5600
 Wire Wire Line
-	12200 3500 11450 3500
-Wire Wire Line
 	12200 3600 11450 3600
 Wire Wire Line
@@
 	5400 10350 4550 10350
 Connection ~ 4550 10350
+Text Notes 9750 3150 0    60   ~ 0
+status went from pin 22 to pin 3\nbuttons to pin 22\nwiz CS to 15
 $EndSCHEMATC
